File: kronos.kicad_pcb (KiCad board)
At the start: 2 copper layers, 104 parts, among them SW1 SW_Push, SW10 SW_Push, SW11 SW_Push, SW12 SW_Push, SW13 SW_Push, SW14 SW_Push, SW15 SW_Push, SW16 SW_Push, SW17 SW_Push, SW18 SW_Push, SW19 SW_Push, SW2 SW_Push, SW20 SW_Push, SW21 SW_Push, SW22 SW_Push, SW23 SW_Push, SW24 SW_Push, SW25 SW_Push, SW26 SW_Push, SW27 SW_Push, SW28 SW_Push, SW29 SW_Push, SW3 SW_Push, SW30 SW_Push, SW31 SW_Push, SW32 SW_Push, SW33 SW_Push, SW34 SW_Push, SW35 SW_Push, SW36 SW_Push, SW37 SW_Push, SW38 SW_Push, SW39 SW_Push, SW4 SW_Push, SW40 SW_Push, SW41 SW_Push, SW42 SW_Push, SW5 SW_Push, SW6 SW_Push, SW7 SW_Push, SW8 SW_Push, SW9 SW_Push, U1 XIAO-nRF52840-SMD, U2 XIAO-nRF52840-SMD

Commit message: PCB akmost done
PCB added; scheme update; blah blah
Parts:
- removed R1, R3: 806K, Resistor_SMD:R_0805_2012Metric
- removed R2, R4: 2M, Resistor_SMD:R_0805_2012Metric
- removed U1, U2: XIAO-nRF52840-SMD, kronoschems:modified-XIAO-nRF52840-SMD
- added D100: WS2812B, LED_SMD:LED_WS2812B_PLCC4_5.0x5.0mm_P3.2mm, F.Cu at (97.4, 101.0)
- added D101: WS2812B, LED_SMD:LED_WS2812B_PLCC4_5.0x5.0mm_P3.2mm, F.Cu at (221.3, 69.3)
- added D102: WS2812B, LED_SMD:LED_WS2812B_PLCC4_5.0x5.0mm_P3.2mm, F.Cu at (59.4, 98.0)
- added D103: WS2812B, LED_SMD:LED_WS2812B_PLCC4_5.0x5.0mm_P3.2mm, F.Cu at (182.3, 69.2)
- added D104: WS2812B, LED_SMD:LED_WS2812B_PLCC4_5.0x5.0mm_P3.2mm, F.Cu at (163.4, 77.5)
- added D105: WS2812B, LED_SMD:LED_WS2812B_PLCC4_5.0x5.0mm_P3.2mm, F.Cu at (59.4, 79.0)
- added D106: WS2812B, LED_SMD:LED_WS2812B_PLCC4_5.0x5.0mm_P3.2mm, F.Cu at (259.9, 122.5)
- added D107: WS2812B, LED_SMD:LED_WS2812B_PLCC4_5.0x5.0mm_P3.2mm, F.Cu at (98.0, 62.5)
- added D108: WS2812B, LED_SMD:LED_WS2812B_PLCC4_5.0x5.0mm_P3.2mm, F.Cu at (39.4, 126.0)
- added D109: WS2812B, LED_SMD:LED_WS2812B_PLCC4_5.0x5.0mm_P3.2mm, F.Cu at (77.9, 127.5)
- added D110: WS2812B, LED_SMD:LED_WS2812B_PLCC4_5.0x5.0mm_P3.2mm, F.Cu at (116.4, 127.5)
- added D111: WS2812B, LED_SMD:LED_WS2812B_PLCC4_5.0x5.0mm_P3.2mm, F.Cu at (59.0, 116.8)
- added D112: WS2812B, LED_SMD:LED_WS2812B_PLCC4_5.0x5.0mm_P3.2mm, F.Cu at (78.4, 89.0)
- added D113: WS2812B, LED_SMD:LED_WS2812B_PLCC4_5.0x5.0mm_P3.2mm, F.Cu at (201.9, 120.7)
- added D114: WS2812B, LED_SMD:LED_WS2812B_PLCC4_5.0x5.0mm_P3.2mm, F.Cu at (182.9, 126.5)
- added D115: WS2812B, LED_SMD:LED_WS2812B_PLCC4_5.0x5.0mm_P3.2mm, F.Cu at (97.4, 81.5)
- added D116: WS2812B, LED_SMD:LED_WS2812B_PLCC4_5.0x5.0mm_P3.2mm, F.Cu at (222.4, 106.2)
- added D117: WS2812B, LED_SMD:LED_WS2812B_PLCC4_5.0x5.0mm_P3.2mm, F.Cu at (201.3, 62.4)
- added D118: WS2812B, LED_SMD:LED_WS2812B_PLCC4_5.0x5.0mm_P3.2mm, F.Cu at (202.4, 82.5)
- added D119: WS2812B, LED_SMD:LED_WS2812B_PLCC4_5.0x5.0mm_P3.2mm, F.Cu at (78.4, 70.0)
- added D120: WS2812B, LED_SMD:LED_WS2812B_PLCC4_5.0x5.0mm_P3.2mm, F.Cu at (115.9, 108.0)
- added D121: WS2812B, LED_SMD:LED_WS2812B_PLCC4_5.0x5.0mm_P3.2mm, F.Cu at (135.4, 116.5)
- added D122: WS2812B, LED_SMD:LED_WS2812B_PLCC4_5.0x5.0mm_P3.2mm, F.Cu at (135.4, 97.2)
- added D123: WS2812B, LED_SMD:LED_WS2812B_PLCC4_5.0x5.0mm_P3.2mm, F.Cu at (116.5, 70.0)
- added D124: WS2812B, LED_SMD:LED_WS2812B_PLCC4_5.0x5.0mm_P3.2mm, F.Cu at (135.4, 78.2)
- added D125: WS2812B, LED_SMD:LED_WS2812B_PLCC4_5.0x5.0mm_P3.2mm, F.Cu at (116.3, 89.0)
- added D126: WS2812B, LED_SMD:LED_WS2812B_PLCC4_5.0x5.0mm_P3.2mm, F.Cu at (182.9, 89.0)
- added D127: WS2812B, LED_SMD:LED_WS2812B_PLCC4_5.0x5.0mm_P3.2mm, F.Cu at (135.4, 135.5)
- added D86: WS2812B, LED_SMD:LED_WS2812B_PLCC4_5.0x5.0mm_P3.2mm, F.Cu at (241.3, 116.3)
- added D87: WS2812B, LED_SMD:LED_WS2812B_PLCC4_5.0x5.0mm_P3.2mm, F.Cu at (163.9, 134.8)
- added D88: WS2812B, LED_SMD:LED_WS2812B_PLCC4_5.0x5.0mm_P3.2mm, F.Cu at (58.9, 136.0)
- added D89: WS2812B, LED_SMD:LED_WS2812B_PLCC4_5.0x5.0mm_P3.2mm, F.Cu at (240.8, 135.3)
- added D90: WS2812B, LED_SMD:LED_WS2812B_PLCC4_5.0x5.0mm_P3.2mm, F.Cu at (221.8, 125.7)
- added D91: WS2812B, LED_SMD:LED_WS2812B_PLCC4_5.0x5.0mm_P3.2mm, F.Cu at (182.9, 107.7)
- added D92: WS2812B, LED_SMD:LED_WS2812B_PLCC4_5.0x5.0mm_P3.2mm, F.Cu at (97.4, 120.5)
- added D93: WS2812B, LED_SMD:LED_WS2812B_PLCC4_5.0x5.0mm_P3.2mm, F.Cu at (221.3, 87.2)
- added D94: WS2812B, LED_SMD:LED_WS2812B_PLCC4_5.0x5.0mm_P3.2mm, F.Cu at (163.8, 97.8)
- added D95: WS2812B, LED_SMD:LED_WS2812B_PLCC4_5.0x5.0mm_P3.2mm, F.Cu at (240.8, 96.3)
- added D96: WS2812B, LED_SMD:LED_WS2812B_PLCC4_5.0x5.0mm_P3.2mm, F.Cu at (78.4, 108.5)
- added D97: WS2812B, LED_SMD:LED_WS2812B_PLCC4_5.0x5.0mm_P3.2mm, F.Cu at (163.9, 116.2)
- added D98: WS2812B, LED_SMD:LED_WS2812B_PLCC4_5.0x5.0mm_P3.2mm, F.Cu at (201.9, 101.3)
- added D99: WS2812B, LED_SMD:LED_WS2812B_PLCC4_5.0x5.0mm_P3.2mm, F.Cu at (240.8, 77.3)
- added U3: Seeeduino Xiao nRF52840, PCM_marbastlib-xp-promicroish:Xiao_nRF52840_ACH, F.Cu at (262.0, 95.0)
- added U4: Seeeduino Xiao nRF52840, PCM_marbastlib-xp-promicroish:Xiao_nRF52840_ACH, F.Cu at (38.4, 99.0)
- D1, D10, D11, D12, D13, D14, D15, D16, D17, D18, D19, D2, D20, D21, D22, D23, D24, D25, D26, D27, D28, D29, D3, D30, D31, D32, D33, D34, D35, D36, D37, D38, D39, D4, D40, D41, D42, D5, D6, D7, D8, D9, SW16: moved to B.Cu
- moved H10 170.3 mm to (140.8, 179.5)
- moved H6 170.3 mm to (140.8, 153.5)
- moved H7 170.3 mm to (140.8, 160.0)
- moved H8 170.3 mm to (140.8, 166.5)
- moved H9 170.3 mm to (140.8, 173.0)
- moved H1 169.5 mm to (29.5, 150.0)
- moved H2 169.5 mm to (29.5, 156.5)
- moved H3 169.5 mm to (29.5, 163.0)
- moved H4 169.5 mm to (29.5, 169.5)
- moved H5 169.5 mm to (29.5, 176.0)
- moved D19 127.7 mm to (48.5, 126.5), turned to -90 degrees
- moved D38 121.2 mm to (172.0, 136.2), turned to -90 degrees
- moved TP3 119.8 mm to (159.6, 184.8)
- moved TP4 119.8 mm to (159.6, 188.8)
- moved D23 109.7 mm to (67.5, 136.2), turned to 90 degrees
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Connections:
- D12 pad 1: unconnected-(D12-K-Pad1) -> Net-(D12-K)
- D18 pad 1: Net-(D18-K) -> Net-(D12-K)
- D21 pad 1: Net-(D18-K) -> Net-(D12-K)
- D33 pad 1: unconnected-(D33-K-Pad1) -> Net-(D25-K)
- D4 pad 1: Net-(D18-K) -> Net-(D12-K)
- D8 pad 1: Net-(D18-K) -> Net-(D12-K)
